Commit message: Changed the Mesh and Link Origins, For Testing Robot Model in Gazebo

File: robot_simulation/URDF/sr_scara_hx.xacro (robot description, xacro)
@@ -13,5 +13,5 @@
 <link name="base_link">
  <visual>
-  <origin xyz="0 0 0.00158925" rpy="0 0 0" />
+  <origin xyz="0 0 0.151" rpy="0 0 0" />
    <geometry>
      <mesh filename="package://robot_simulation/meshes/base_R01.stl" scale="0.001 0.001 0.001"/>
@@ -20,5 +20,5 @@
  </visual>
  <collision>
-  <origin xyz="0 0 0.00158925" rpy="0 0 0" />
+  <origin xyz="0 0 0.151" rpy="0 0 0" />
    <geometry>
      <mesh filename="package://robot_simulation/meshes/base_R01.stl" scale="0.001 0.001 0.001"/>
@@ -26,5 +26,5 @@
  </collision>
  <inertial>
-      <origin xyz="0 0 0.00158925" rpy="0 0 0"/>
+      <origin xyz="0 0 0.151" rpy="0 0 0"/>
       <mass value="30.0"/>
       <inertia
@@ -36,5 +36,5 @@
 <link name="link1">
  <visual>
-  <origin xyz="0 0 0" rpy="0 0 0" />
+  <origin xyz="-0.18 0 0.365" rpy="0 0 0" />
    <geometry>
      <mesh filename="package://robot_simulation/meshes/arm_link_R01.stl" scale="0.001 0.001 0.001"/>
@@ -43,5 +43,5 @@
  </visual>
  <collision>
-  <origin xyz="0 0 0" rpy="0 0 0" />
+  <origin xyz="-0.18 0 0.365" rpy="0 0 0" />
    <geometry>
      <mesh filename="package://robot_simulation/meshes/arm_link_R01.stl" scale="0.001 0.001 0.001"/>
@@ -49,5 +49,5 @@
  </collision>
  <inertial>
-      <origin xyz="0 0 0" rpy="0 0 0"/>
+      <origin xyz="-0.18 0 0.365" rpy="0 0 0"/>
       <mass value="10.0"/>
       <inertia
@@ -59,5 +59,5 @@
 <link name="link2">
  <visual>
-  <origin xyz="0.300 0 0" rpy="0 0 0" />
+  <origin xyz="-0.25 0 0.47" rpy="0 0 0" />
    <geometry>
      <mesh filename="package://robot_simulation/meshes/head_link_R01.stl" scale="0.001 0.001 0.001"/>
@@ -66,5 +66,5 @@
  </visual>
  <collision>
-  <origin xyz="0.300 0 0" rpy="0 0 0" />
+  <origin xyz="-0.25 0 0.47" rpy="0 0 0" />
    <geometry>
      <mesh filename="package://robot_simulation/meshes/head_link_R01.stl" scale="0.001 0.001 0.001"/>
@@ -72,5 +72,5 @@
   </collision>
  <inertial>
-      <origin xyz="0.300 0 0" rpy="0 0 0"/>
+      <origin xyz="-0.25 0 0.47" rpy="0 0 0"/>
       <mass value="10.0"/>
       <inertia
@@ -82,5 +82,5 @@
 <link name="probe">
  <visual>
-  <origin xyz="-0.65 0 0.43" rpy="0 0 0" />
+  <origin xyz="-0.7 0 0.43" rpy="0 0 0" />
   <geometry>
      <mesh filename="package://robot_simulation/meshes/End_link_R01.stl" scale="0.001 0.001 0.001"/>
@@ -89,5 +89,5 @@
  </visual>
  <collision>
-  <origin xyz="-0.65 0 0.43" rpy="0 0 0" />
+  <origin xyz="-0.7 0 0.43" rpy="0 0 0" />
   <geometry>
      <mesh filename="package://robot_simulation/meshes/End_link_R01.stl" scale="0.001 0.001 0.001"/>
@@ -95,5 +95,5 @@
  </collision>
  <inertial>
-      <origin xyz="-0.65 0 0.43" rpy="0 0 0"/>
+      <origin xyz="-0.7 0 0.43" rpy="0 0 0"/>
       <mass value="2.0"/>
       <inertia
@@ -105,5 +105,5 @@
 <link name="gripper">
  <visual>
-  <origin xyz="0 0 0" rpy="0 0 0"/>
+  <origin xyz="-0.05 0 0" rpy="0 0 0"/>
   <geometry>
   <cylinder length="0.08" radius="0.04"/>
@@ -112,5 +112,5 @@
  </visual>
  <collision>
-  <origin xyz="0 0 0" rpy="0 0 0"/>
+  <origin xyz="-0.05 0 0" rpy="0 0 0"/>
   <geometry>
   <cylinder length="0.08" radius="0.04"/>
@@ -118,5 +118,5 @@
  </collision>
  <inertial>
-     <origin xyz="0 0 0" rpy="0 0 0"/>
+     <origin xyz="-0.05 0 0" rpy="0 0 0"/>
      <mass value="0.3"/>
      <inertia
@@ -128,5 +128,5 @@
 <link name="gripper_end_effector">
  <visual>
-  <origin xyz="0 0 0" rpy="0 0 0"/>
+  <origin xyz="-0.04 0 -0.01" rpy="0 0 0"/>
   <geometry>
   <cylinder length="0.04" radius="0.02"/>
@@ -135,5 +135,5 @@
  </visual>
  <collision>
-  <origin xyz="0 0 0" rpy="0 0 0"/>
+  <origin xyz="-0.04 0 -0.01" rpy="0 0 0"/>
   <geometry>
   <cylinder length="0.001" radius="0.004"/>
@@ -141,5 +141,5 @@
  </collision>
  <inertial>
-     <origin xyz="0 0 0" rpy="0 0 0"/>
+     <origin xyz="-0.04 0 -0.01" rpy="0 0 0"/>
      <mass value="0.1"/>
      <inertia
