Commit message: Changed the joint offset

File: robot_simulation/URDF/sr_scara_hx.urdf (robot description, URDF)
Before this commit: robot sr_scara_hx, 6 links, 5 joints
Joints:
- joint joint1: origin xyz=0 0 0.00158925 rpy=0 0 0 -> xyz=0 0 0.003 rpy=0 0 0
- joint joint2: origin xyz=-0.3 0 0 rpy=0 0 0 -> xyz=-0.3 0 0.006 rpy=0 0 0

File: robot_simulation/URDF/sr_scara_hx.xacro (robot description, xacro)
@@ -153,5 +153,5 @@
   <axis xyz="0 0 1" />
   <limit effort="3.0" velocity="0.01" lower="-2.792" upper="2.792"/>
-  <origin xyz="0 0 0.00158925" rpy="0 0 0" />
+  <origin xyz="0 0 0.003" rpy="0 0 0" />
   <parent link="base_link" />
   <child link="link1" />
@@ -160,5 +160,5 @@
  <axis xyz="0 0 1" />
  <limit effort="3.0" velocity="0.01" lower="-2.443" upper="2.443"/>
- <origin xyz="-0.3 0 0" rpy="0 0 0" />
+ <origin xyz="-0.3 0 0.006" rpy="0 0 0" />
  <parent link="link1" />
  <child link="link2" />
